Commit message: changed path and commented lidar , cam, depth cam.

File: description/thar.urdf.xacro (robot description, xacro)
@@ -4,6 +4,6 @@
     <xacro:include filename="thar3_core.xacro" />
     <xacro:include filename="gazebo_control.xacro"/>
-    <xacro:include filename="lidar.xacro" />
-    <xacro:include filename="depth_camera.xacro" />
+    <!-- <xacro:include filename="lidar.xacro" /> -->
+    <!-- <xacro:include filename="depth_camera.xacro" /> -->
     <!-- <xacro:include filename="camera.xacro" /> -->
 </robot>

File: description/thar3_core.xacro (robot description, xacro)
@@ -51,5 +51,5 @@
       <geometry>
         <mesh
-          filename="file:///home/rozy/thar_ws/src/thar_bot/meshes/chassisblender.dae" />
+          filename="file:///home/mahindra/thar_ws/src/thar_bot/meshes/chassisblender.dae" />
       </geometry>
       <material name="gray"/>
@@ -61,5 +61,5 @@
       <geometry>
         <mesh
-          filename="file:///home/rozy/thar_ws/src/thar_bot/meshes/base_link.STL" />
+          filename="file:///home/mahindra/thar_ws/src/thar_bot/meshes/base_link.STL" />
       </geometry>
     </collision>
@@ -109,5 +109,5 @@
       <geometry>
         <mesh
-          filename="file:///home/rozy/thar_ws/src/thar_bot/meshes/wheelblender.dae" />
+          filename="file:///home/mahindra/thar_ws/src/thar_bot/meshes/wheelblender.dae" />
       </geometry>
       <material
@@ -123,5 +123,5 @@
       <geometry>
         <mesh
-          filename="file:///home/rozy/thar_ws/src/thar_bot/meshes/front_left_wheel.STL" />
+          filename="file:///home/mahindra/thar_ws/src/thar_bot/meshes/front_left_wheel.STL" />
       </geometry>
     </collision>
@@ -177,5 +177,5 @@
       <geometry>
         <mesh
-          filename="file:///home/rozy/thar_ws/src/thar_bot/meshes/wheelblender.dae" />
+          filename="file:///home/mahindra/thar_ws/src/thar_bot/meshes/wheelblender.dae" />
       </geometry>
       <material
@@ -191,5 +191,5 @@
       <geometry>
         <mesh
-          filename="file:///home/rozy/thar_ws/src/thar_bot/meshes/front_right_wheel.STL" />
+          filename="file:///home/mahindra/thar_ws/src/thar_bot/meshes/front_right_wheel.STL" />
       </geometry>
     </collision>
@@ -245,5 +245,5 @@
       <geometry>
         <mesh
-          filename="file:///home/rozy/thar_ws/src/thar_bot/meshes/wheelblender.dae" />
+          filename="file:///home/mahindra/thar_ws/src/thar_bot/meshes/wheelblender.dae" />
       </geometry>
       <material
@@ -259,5 +259,5 @@
       <geometry>
         <mesh
-          filename="file:///home/rozy/thar_ws/src/thar_bot/meshes/back_left_wheel.STL" />
+          filename="file:///home/mahindra/thar_ws/src/thar_bot/meshes/back_left_wheel.STL" />
       </geometry>
     </collision>
@@ -313,5 +313,5 @@
       <geometry>
         <mesh
-          filename="file:///home/rozy/thar_ws/src/thar_bot/meshes/wheelblender.dae" />
+          filename="file:///home/mahindra/thar_ws/src/thar_bot/meshes/wheelblender.dae" />
       </geometry>
       <material
@@ -320,14 +320,14 @@
           rgba="0.792156862745098 0.819607843137255 0.933333333333333 1" /> -->
         <texture
-          filename="file:///home/rozy/thar_ws/src/thar_bot/textures/Wheel.dae" />
-      </material>
-    </visual>
-    <collision>
-      <origin
-        xyz="0 0 0"
-        rpy="0 0 0" />
-      <geometry>
-        <mesh
-          filename="file:///home/rozy/thar_ws/src/thar_bot/meshes/back_right_wheel.STL" />
+          filename="file:///home/mahindra/thar_ws/src/thar_bot/textures/Wheel.dae" />
+      </material>
+    </visual>
+    <collision>
+      <origin
+        xyz="0 0 0"
+        rpy="0 0 0" />
+      <geometry>
+        <mesh
+          filename="file:///home/mahindra/thar_ws/src/thar_bot/meshes/back_right_wheel.STL" />
       </geometry>
     </collision>
@@ -369,5 +369,5 @@
       <geometry>
         <mesh
-          filename="file:///home/rozy/thar_ws/src/thar_bot/meshes/wheelblender.dae" />
+          filename="file:///home/mahindra/thar_ws/src/thar_bot/meshes/wheelblender.dae" />
       </geometry>
       <material
@@ -376,14 +376,14 @@
           rgba="0.79216 0.81961 0.93333 1" />
         <texture
-          filename="file:///home/rozy/thar_ws/src/thar_bot/meshes/wheelblender.dae" />
-      </material>
-    </visual>
-    <collision>
-      <origin
-        xyz="0 0 0"
-        rpy="0 0 0" />
-      <geometry>
-        <mesh
-          filename="file:///home/rozy/thar_ws/src/thar_bot/meshes/wheelblender.dae" />
+          filename="file:///home/mahindra/thar_ws/src/thar_bot/meshes/wheelblender.dae" />
+      </material>
+    </visual>
+    <collision>
+      <origin
+        xyz="0 0 0"
+        rpy="0 0 0" />
+      <geometry>
+        <mesh
+          filename="file:///home/mahindra/thar_ws/src/thar_bot/meshes/wheelblender.dae" />
       </geometry>
     </collision>
