Commit message: recent

File: description/thar3_core.xacro (robot description, xacro)
@@ -315,11 +315,11 @@
           filename="file:///home/mahindra/thar_ws/src/thar_bot/meshes/wheelblender.dae" />
       </geometry>
-      <material
+      <!-- <material
         name="">
-        <!-- <color
-          rgba="0.792156862745098 0.819607843137255 0.933333333333333 1" /> -->
+        <color
+          rgba="0.792156862745098 0.819607843137255 0.933333333333333 1" />
         <texture
           filename="file:///home/mahindra/thar_ws/src/thar_bot/textures/Wheel.dae" />
-      </material>
+      </material> -->
     </visual>
     <collision>
@@ -371,5 +371,5 @@
           filename="file:///home/mahindra/thar_ws/src/thar_bot/meshes/wheelblender.dae" />
       </geometry>
-      <material
+      <!-- <material
         name="wheel">
         <color
@@ -377,5 +377,5 @@
         <texture
           filename="file:///home/mahindra/thar_ws/src/thar_bot/meshes/wheelblender.dae" />
-      </material>
+      </material> -->
     </visual>
     <collision>
